Commit message: Box cannot have same name as built-in macro

File: objects/open_box.urdf.xacro (robot description, xacro)
@@ -1,4 +1,4 @@
 <?xml version="1.0"?>
-<robot name="table" xmlns:xacro="http://wiki.ros.org/xacro">
+<robot name="open_box" xmlns:xacro="http://wiki.ros.org/xacro">
   <xacro:arg name="prefix" default="box_"/>
   <xacro:arg name="connected_to" default=""/>
@@ -10,7 +10,7 @@
   <xacro:arg name="wall_thickness" default="0.02"/>
   <xacro:arg name="mass" default="3.0"/>
-  <xacro:include filename="$(find object_descriptions)/objects/box.xacro"/>
-  <xacro:box prefix="$(arg prefix)" connected_to="$(arg connected_to)" xyz="$(arg xyz)" rpy="$(arg rpy)"
-             height="$(arg height)" x_size="$(arg x_size)" y_size="$(arg y_size)" thickness="$(arg wall_thickness)"
-             mass="$(arg mass)"/>
+  <xacro:include filename="$(find object_descriptions)/objects/open_box.xacro"/>
+  <xacro:open_box prefix="$(arg prefix)" connected_to="$(arg connected_to)" xyz="$(arg xyz)" rpy="$(arg rpy)"
+                  height="$(arg height)" x_size="$(arg x_size)" y_size="$(arg y_size)" thickness="$(arg wall_thickness)"
+                  mass="$(arg mass)"/>
 </robot>

File: objects/open_box.xacro (robot description, xacro)
@@ -1,5 +1,5 @@
 <?xml version="1.0"?>
 <robot name="box" xmlns:xacro="http://wiki.ros.org/xacro">
-  <xacro:macro name="box"
+  <xacro:macro name="open_box"
                params="prefix='box_' connected_to:='' xyz:='0 0 0' rpy:='0 0 0' height:=0.15 x_size:=0.5 y_size=0.5
                thickness=0.02 mass=3.0">
