Commit message: Handle odom explicitely

File: objects/open_box.xacro (robot description, xacro)
@@ -14,4 +14,8 @@
       <xacro:property name="base_frame_name" value="${connected_to}"/>
     </xacro:unless>
+    <xacro:if value="${connected_to == 'odom'}">
+      <link name="odom"/>
+      <xacro:property name="base_frame_name" value="odom"/>
+    </xacro:if>
     <joint name="${prefix}base_to_${base_frame_name}" type="fixed">
       <parent link="${base_frame_name}"/>

File: objects/soccerball.xacro (robot description, xacro)
@@ -11,4 +11,8 @@
       <xacro:property name="base_frame_name" value="${connected_to}"/>
     </xacro:unless>
+    <xacro:if value="${connected_to == 'odom'}">
+      <link name="odom"/>
+      <xacro:property name="base_frame_name" value="odom"/>
+    </xacro:if>
     <joint name="ball_to_${base_frame_name}" type="fixed">
       <parent link="${base_frame_name}"/>

File: objects/table.xacro (robot description, xacro)
@@ -19,4 +19,8 @@
       <xacro:property name="base_frame_name" value="${connected_to}"/>
     </xacro:unless>
+    <xacro:if value="${connected_to == 'odom'}">
+      <link name="odom"/>
+      <xacro:property name="base_frame_name" value="odom"/>
+    </xacro:if>
     <joint name="${prefix}base_to_${base_frame_name}" type="fixed">
       <parent link="${base_frame_name}"/>
